File: IntrusionNode_v2/IntrusionNode_v2.sch (EAGLE design)
At the start: 38 parts, among them IC1 MCP1703CB, Q1 MOSFET-PCHANNELSMD, U1 RFM69, U2 MCP73831, U3 ATMEGA328P-AU, U4 MMA8452Q, Y1 16MHZ

Commit message: *** Parts order place on Digikey
Web ID    149351856     Access ID    51215     Salesorder Number    43979223     Submitted    8/25/2015 4:06:46 PM

Modified board, adding notch, also changed part numbers for diode
and MOSFET to reduce current.
Parts:
- D1: value SCHOTTKY -> BAT20J; device SparkFun-DiscreteSemi:DIODESOD123 -> SparkFun-DiscreteSemi:DIODE-SCHOTTKY-BAT20J; PARTNO B130LAW-7-F -> BAT20JFILM
- Q1: PARTNO SSM3J328R,LF -> PMV48XP,215
- R7: value 10K -> 100K; PARTNO RC2012J103CS -> RC2012J104CS
- R8: value 3.3M -> 10M; PARTNO RC2012F335CS -> RC2012F106CS
- R9: value 5.36M -> 10M; PARTNO RC2012F5364CS -> RC2012F106CS
Changed lines of the file:
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@@
 <part name="GND9" library="supply2" deviceset="GND" device=""/>
 <part name="Q1" library="SparkFun-DiscreteSemi" deviceset="MOSFET-PCHANNEL" device="SMD">
-<attribute name="PARTNO" value="SSM3J328R,LF"/>
+<attribute name="PARTNO" value="PMV48XP,215"/>
 </part>
-<part name="D1" library="SparkFun-DiscreteSemi" deviceset="DIODE" device="SOD123" value="SCHOTTKY">
-<attribute name="PARTNO" value="B130LAW-7-F"/>
+<part name="D1" library="SparkFun-DiscreteSemi" deviceset="DIODE-SCHOTTKY" device="-BAT20J" value="BAT20J">
+<attribute name="PARTNO" value="BAT20JFILM"/>
 </part>
-<part name="R7" library="rcl" deviceset="R-US_" device="R0805" value="10K">
-<attribute name="PARTNO" value="RC2012J103CS"/>
+<part name="R7" library="rcl" deviceset="R-US_" device="R0805" value="100K">
+<attribute name="PARTNO" value="RC2012J104CS"/>
 </part>
 <part name="C9" library="rcl" deviceset="C-US" device="C0805" value="1u">
@@
 <attribute name="PARTNO" value="629105136821"/>
 </part>
-<part name="R8" library="rcl" deviceset="R-US_" device="R0805" value="3.3M">
-<attribute name="PARTNO" value="RC2012F335CS"/>
+<part name="R8" library="rcl" deviceset="R-US_" device="R0805" value="10M">
+<attribute name="PARTNO" value="RC2012F106CS"/>
 </part>
-<part name="R9" library="rcl" deviceset="R-US_" device="R0805" value="5.36M">
-<attribute name="PARTNO" value="RC2012F5364CS"/>
+<part name="R9" library="rcl" deviceset="R-US_" device="R0805" value="10M">
+<attribute name="PARTNO" value="RC2012F106CS"/>
 </part>
 <part name="C10" library="rcl" deviceset="C-US" device="C0805" value="0.1u">
